File: PCB/PowerUnit.kicad_pcb (KiCad board)
At the start: 2 copper layers, 116 parts, among them J1 MX150-20, J2 MX150-20, J3 MX150-8, J4 REDCUBE, J5 CON-3, Q1 BC847C, Q10 STD45P4LLF6AG, Q11 STD45P4LLF6AG, Q12 STD15P6F6AG, Q13 STD15P6F6AG, Q2 STD15P6F6AG, Q3 STD45P4LLF6AG, Q4 STD45P4LLF6AG, Q5 STD15P6F6AG, Q6 STD15P6F6AG, Q7 STD45P4LLF6AG, Q8 BC847C, Q9 STD15P6F6AG, U1 STM8S001J3M3, U2 L5150BN

Commit message: First PCB Layout done
Parts:
- removed D16, D18: SMA6F15AY, erp:D_SMA
- added D38: SMA6F15AY, erp:D_SMA, F.Cu at (132.0, 122.5)
- added D39: LL4148, erp:D_MiniMELF, F.Cu at (137.5, 89.0)
- added D40: RED, erp:LED_0805_2012Metric, F.Cu at (134.0, 90.0)
- added D41: LL4148, erp:D_MiniMELF, F.Cu at (198.0, 89.0)
- added D42: RED, erp:LED_0805_2012Metric, F.Cu at (201.5, 90.0)
- added D43: SMA6F15AY, erp:D_SMA, F.Cu at (198.5, 122.5)
- added F4: FUSE, erp:Keystone_FuseHolder, F.Cu at (176.0, 103.0)
- added F7: FUSE, erp:Keystone_FuseHolder, F.Cu at (134.0, 103.0)
- added G***: LOGO, test:Untitled, F.Cu at (209.5, 112.5)
- added J10: MH_M4, erp:MountingHole_4.3mm_M4_Pad_Via, F.Cu at (90.0, 143.5)
- added J11: MH_M4, erp:MountingHole_4.3mm_M4_Pad_Via, F.Cu at (155.0, 90.0)
- added J12: MH_M4, erp:MountingHole_4.3mm_M4_Pad_Via, F.Cu at (155.0, 143.5)
- added J13: MH_M4, erp:MountingHole_4.3mm_M4_Pad_Via, F.Cu at (90.0, 90.0)
- added J6: MH_M4, erp:MountingHole_4.3mm_M4_Pad_Via, F.Cu at (55.0, 135.0)
- added J7: MH_M4, erp:MountingHole_4.3mm_M4_Pad_Via, F.Cu at (55.0, 90.0)
- added J8: MH_M4, erp:MountingHole_4.3mm_M4_Pad_Via, F.Cu at (210.0, 90.0)
- added J9: MH_M4, erp:MountingHole_4.3mm_M4_Pad_Via, F.Cu at (210.0, 135.0)
- added R37: 2.2k, erp:R_0805_2012Metric, F.Cu at (134.0, 87.5)
- added R38: 2.2k, erp:R_0805_2012Metric, F.Cu at (201.5, 87.5)
- added R39: 2.2k, erp:R_0805_2012Metric, F.Cu at (94.5, 117.5)
- moved C2 178.1 mm to (60.0, 97.0), turned to 90 degrees
- moved R1 170.8 mm to (61.0, 104.0), turned to 180 degrees
- moved R22 157.5 mm to (54.0, 126.5), turned to 270 degrees
- moved C7 157.4 mm to (56.5, 122.5), turned to 90 degrees
- moved R16 151.9 mm to (66.0, 117.5)
- moved R4 143.0 mm to (65.0, 101.0), turned to 270 degrees
- moved R2 141.8 mm to (60.0, 101.0), turned to 270 degrees
- moved R11 140.1 mm to (56.5, 126.6), turned to 270 degrees
- moved C1 139.9 mm to (69.0, 87.0)
- moved R27 139.9 mm to (75.5, 117.5)
- moved J5 139.7 mm to (74.0, 88.0), turned to 90 degrees
- moved D2 134.5 mm to (67.5, 100.0), turned to 270 degrees
- moved R5 134.4 mm to (78.0, 98.0), turned to 90 degrees
- moved C11 133.6 mm to (54.0, 122.5), turned to 90 degrees
- moved R13 133.4 mm to (73.0, 98.0), turned to 90 degrees
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- renumbered F4 to F10, F7 to F9
Connections:
- F1 pad 2A: /PWD_ECU -> /PWD_START
- F1 pad 2B: /PWD_ECU -> /PWD_START
- F2 pad 2A: /PWD_INJECT -> /PWD_ECU
- F2 pad 2B: /PWD_INJECT -> /PWD_ECU
- F6 pad 2A: /PWD_LIGHT -> /PWD_AUX
- F6 pad 2B: /PWD_LIGHT -> /PWD_AUX
- F8 pad 2A: /PWD_AUX -> /PWD_LIGHT
- F8 pad 2B: /PWD_AUX -> /PWD_LIGHT
- J1 pad 1: (no net) -> GND
- J1 pad 11: GND -> (no net)
- J1 pad 14: /IN_INJECT -> /IN_FAN_A
- J1 pad 15: /IN_FAN_A -> /IN_INJECT
- J1 pad 18: /OUT_LIGHT -> /START
- J1 pad 19: (no net) -> /START
- J1 pad 6: /PWD_ECU -> /OUT_LIGHT
- J1 pad 7: /START -> /PWD_ECU
- J1 pad 8: /START -> /PWD_ECU
- J1 pad 9: /PWD_FAN -> /PWD_START
- J2 pad 1: (no net) -> GND
- J2 pad 11: GND -> (no net)
- J2 pad 14: /START -> /IN_RAIN
- J2 pad 15: /IN_FAN_B -> /IN_FUEL
- J2 pad 16: /IN_RAIN -> /IN_LIGHT
- J2 pad 17: /IN_FUEL -> /IN_FAN_B
- J2 pad 18: /IN_LIGHT -> /IN_IGN
- J2 pad 19: /IN_IGN -> /START
- J2 pad 2: /PWD_AUX -> /OUT_LEFT
- J2 pad 3: /OUT_LIGHT -> /OUT_RIGHT
- J2 pad 4: /PWD_ECU -> /OUT_LIGHT
- J2 pad 5: /OUT_AUX -> /IN_AUX
- J2 pad 6: /IN_AUX -> /PWD_DASH
- J2 pad 7: /PWD_MISC -> /PWD_DASH
- J2 pad 8: /OUT_LEFT -> /PWD_AUX
- J2 pad 9: /OUT_RIGHT -> /OUT_AUX
- J3 pad 1: /OUT_LIGHT -> GND
- J3 pad 2: /OUT_LEFT -> /OUT_RAIN
- J3 pad 3: /OUT_RIGHT -> /OUT_BRAKE_B
- J3 pad 4: /OUT_RAIN -> /OUT_FUEL
- J3 pad 5: GND -> /OUT_LIGHT
- J3 pad 6: /OUT_BRAKE_A -> /OUT_LEFT
- J3 pad 7: /OUT_BRAKE_B -> /OUT_RIGHT
- J3 pad 8: /OUT_FUEL -> /OUT_BRAKE_A
- R1 pad 1: /PWD_LIGHT -> +5V
- R3 pad 1: /PWD_LIGHT -> +5V
Routing:
- net /OUT_LIGHT: track 0.00 -> 151.1 mm, vias 0 -> 12
- net /OUT_RIGHT: track 0.00 -> 148.6 mm, vias 0 -> 10
- net GND: track 0.00 -> 145.9 mm, vias 0 -> 66
- net /OUT_LEFT: track 0.00 -> 142.3 mm, vias 0 -> 10
- net /IN_RIGHT: track 0.00 -> 104.2 mm, vias 0 -> 1
- net /IN_LEFT: track 0.00 -> 101.3 mm, vias 0 -> 1
- net Net-(C13-Pad1): track 0.00 -> 95.8 mm, vias 0 -> 3
- net /IN_FUEL: track 0.00 -> 78.2 mm, vias 0 -> 1
- net /IN_RAIN: track 0.00 -> 71.3 mm, vias 0 -> 1
- net /CAN_H: track 0.00 -> 71.2 mm
- net /START: track 0.00 -> 66.7 mm
- net /CAN_L: track 0.00 -> 66.7 mm
- net +12V: track 0.00 -> 65.9 mm, vias 0 -> 2
- net Net-(Q8-Pad3): track 0.00 -> 54.9 mm, vias 0 -> 2
- net Net-(C10-Pad1): track 0.00 -> 46.5 mm, vias 0 -> 2
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- added copper zone on B.Cu, net +12V
- added copper zone on F.Cu, net +12V
- added copper zone on In1.Cu, net +5V
- added copper zone on B.Cu, net /OUT_AUX
- added copper zone on F.Cu, net /OUT_AUX
- added copper zone on B.Cu, net /OUT_BRAKE_A
- added copper zone on F.Cu, net /OUT_BRAKE_A
- added copper zone on B.Cu, net /OUT_BRAKE_B
- added copper zone on F.Cu, net /OUT_BRAKE_B
- added copper zone on B.Cu, net /OUT_FAN
- added copper zone on F.Cu, net /OUT_FAN
- added copper zone on B.Cu, net /OUT_FUEL
- added copper zone on F.Cu, net /OUT_FUEL
- added copper zone on B.Cu, net /OUT_IGN
- added copper zone on F.Cu, net /OUT_IGN
- added copper zone on B.Cu, net /OUT_INJECT
- added copper zone on F.Cu, net /OUT_INJECT
- added copper zone on B.Cu, net /OUT_LEFT
- added copper zone on F.Cu, net /OUT_LEFT
- added copper zone on B.Cu, net /OUT_LIGHT
- added copper zone on F.Cu, net /OUT_LIGHT
- added copper zone on B.Cu, net /OUT_RAIN
- added copper zone on F.Cu, net /OUT_RAIN
- added copper zone on B.Cu, net /OUT_RIGHT
- added copper zone on F.Cu, net /OUT_RIGHT
- added copper zone on B.Cu, net /PWD_AUX
- added copper zone on F.Cu, net /PWD_AUX
- added copper zone on B.Cu, net /PWD_DASH
- added copper zone on F.Cu, net /PWD_DASH
- added copper zone on B.Cu, net /PWD_ECU
- added copper zone on F.Cu, net /PWD_ECU
- added copper zone on B.Cu, net /PWD_FAN
- added copper zone on F.Cu, net /PWD_FAN
- added copper zone on B.Cu, net /PWD_FUEL
- added copper zone on F.Cu, net /PWD_FUEL
- added copper zone on B.Cu, net /PWD_IGN
- added copper zone on F.Cu, net /PWD_IGN
- added copper zone on B.Cu, net /PWD_INJECT
- added copper zone on F.Cu, net /PWD_INJECT
- added copper zone on B.Cu, net /PWD_LIGHT
- added copper zone on F.Cu, net /PWD_LIGHT
- added copper zone on B.Cu, net /PWD_MISC
- added copper zone on F.Cu, net /PWD_MISC
- added copper zone on B.Cu, net /PWD_START
- added copper zone on F.Cu, net /PWD_START
- added copper zone on In2.Cu, net GND
Other:
- board outline added: 165 x 67.6 mm
- copper layers 2 -> 4
- net class Default: trace_width 0.25 -> 0.3
- net class Output added: clearance 0.2, trace_width 0.8, via_dia 1.3, via_drill 0.7
- board text added: "110000"

Commit message: Now with first Gerber
Parts:
- removed J10, J11, J12, J13, J6, J7, J8, J9: MH_M4, erp:MountingHole_4.3mm_M4_Pad_Via
- added FID1: FIDU, erp:Fiducial_1mm_Mask2mm, F.Cu at (51.5, 95.0)
- added FID2: FIDU, erp:Fiducial_1mm_Mask2mm, F.Cu at (213.5, 140.5)
- added H1: MH_M4, erp:MountingHole_4.3mm_M4_Pad_Via, F.Cu at (55.0, 90.0)
- added H2: MH_M4, erp:MountingHole_4.3mm_M4_Pad_Via, F.Cu at (55.0, 135.0)
- added H3: MH_M4, erp:MountingHole_4.3mm_M4_Pad_Via, F.Cu at (90.0, 90.0)
- added H4: MH_M4, erp:MountingHole_4.3mm_M4_Pad_Via, F.Cu at (90.0, 143.5)
- added H5: MH_M4, erp:MountingHole_4.3mm_M4_Pad_Via, F.Cu at (155.0, 90.0)
- added H6: MH_M4, erp:MountingHole_4.3mm_M4_Pad_Via, F.Cu at (155.0, 143.5)
- added H7: MH_M4, erp:MountingHole_4.3mm_M4_Pad_Via, F.Cu at (210.0, 90.0)
- added H8: MH_M4, erp:MountingHole_4.3mm_M4_Pad_Via, F.Cu at (210.0, 135.0)
