File: PCB/PowerUnit.kicad_pcb (KiCad board)
At the start: 4 copper layers, 165 x 67.6 mm, 120 parts, among them J1 MX150-20, J2 MX150-20, J3 MX150-8, J4 REDCUBE, J5 REDFIT-4, Q1 BC847C, Q2 BC847C, U1 STM8S001J3M3, U10 BTS6143D, U11 BTS6143D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

Commit message: Updated to KiCAD 7.0
Other:
- net class Default removed
- net class Output removed

Commit message: Production data Rev C
Parts:
- removed G***: LOGO, test:Untitled
- added C5: 100n, erp:C_0805_2012Metric, F.Cu at (151.0, 118.0)
- added Q3: BC847C, erp:SOT-23, F.Cu at (155.8, 121.0)
- added R14: 1k, erp:R_0805_2012Metric, F.Cu at (160.5, 128.0)
- added R15: 1k, erp:R_0805_2012Metric, F.Cu at (155.8, 125.5)
- added R8: 1k, erp:R_0805_2012Metric, F.Cu at (160.5, 118.0)
- D10, D11, D12, D13, D14, D15, D17, D28, D29, D3, D38, D4, D43, D5, D6, D7: value SMA6F15AY -> SM6F15AY; footprint erp:D_SMA -> erp:D_SOD-128
- moved R17 2.50 mm to (160.5, 125.5)
- moved R21 2.50 mm to (160.5, 120.5)
- moved R9 2.50 mm to (160.5, 123.0)
- moved D28 2.00 mm to (154.9, 113.0), turned to 0 degrees
- moved D16 1.00 mm to (151.5, 133.0)
- moved D18 1.00 mm to (151.5, 130.5)
- moved D8 1.00 mm to (160.0, 133.0)
- moved D9 1.00 mm to (160.0, 130.5)
Connections:
- J1 pad 11: Net-(J1-Pad11) -> unconnected-(J1-Pin_11-Pad11)
- J1 pad 12: Net-(J1-Pad12) -> /IN_FAN_P
- J2 pad 11: Net-(J2-Pad11) -> unconnected-(J2-Pin_11-Pad11)
- J5 pad 4: Net-(J5-Pad4) -> unconnected-(J5-Pin_4-Pad4)
- U10 pad 4: Net-(U10-Pad4) -> unconnected-(U10-IS-Pad4)
- U11 pad 4: Net-(U11-Pad4) -> unconnected-(U11-IS-Pad4)
- U12 pad 4: Net-(U12-Pad4) -> unconnected-(U12-IS-Pad4)
- U13 pad 4: Net-(U13-Pad4) -> unconnected-(U13-IS-Pad4)
- U3 pad 4: Net-(U3-Pad4) -> unconnected-(U3-IS-Pad4)
- U4 pad 4: Net-(U4-Pad4) -> unconnected-(U4-IS-Pad4)
- U5 pad 4: Net-(U5-Pad4) -> unconnected-(U5-IS-Pad4)
- U6 pad 4: Net-(U6-Pad4) -> unconnected-(U6-IS-Pad4)
- U7 pad 4: Net-(U7-Pad4) -> unconnected-(U7-IS-Pad4)
- U8 pad 4: Net-(U8-Pad4) -> unconnected-(U8-IS-Pad4)
- U9 pad 4: Net-(U9-Pad4) -> unconnected-(U9-IS-Pad4)
Routing:
- net /IN_FAN_P: track 0.00 -> 38.1 mm, vias 0 -> 1
- net Net-(D8-A): track 6.05 -> 20.3 mm
- net Net-(Q3-B): track 0.00 -> 9.31 mm
- net /PWD_FAN: track 20.1 -> 24.6 mm
- net GND: track 133.4 -> 137.4 mm, vias 56 -> 59
- net /IN_FAN_A: track 35.2 -> 32.1 mm
- net /IN_IGN: track 42.5 -> 45.0 mm
- net /IN_BRAKE: track 38.4 -> 36.1 mm
- net /IN_INJECT: track 42.9 -> 44.5 mm
- net Net-(U4-IN): track 29.5 -> 30.5 mm
- net Net-(U3-IN): track 19.4 -> 20.3 mm
Other:
- rule solder_mask_min_width: 0.25 -> 0.2
- board text added: "Prod. 110000 Rev. C"
- board text removed: "Prod. 110000 Rev. B"

Commit message: Update Silkscreen design
Other:
- board text added: "2025-01-13 Revision C"
- board text added: "https://github.com/ JacobNeergaard/powerunit/"
- board text removed: "Prod. 110000 Rev. C"
