File: PCB/PowerUnit.sch (KiCad schematic (older format))
At the start: 115 parts, among them J1 MX150-20, J2 MX150-20, J3 MX150-8, J4 REDCUBE, Q1 BC847C, Q10 STD45P4LLF6AG, Q11 STD45P4LLF6AG, Q12 STD15P6F6AG, Q13 STD15P6F6AG, Q2 STD15P6F6AG, Q3 STD45P4LLF6AG, Q4 STD45P4LLF6AG, Q5 STD15P6F6AG, Q6 STD15P6F6AG, Q7 STD45P4LLF6AG, Q8 BC847C, Q9 STD15P6F6AG, U1 STM8S001J3M3, U2 L5150BN

Commit message: Added SWIM connector
Parts:
- added J5: CON-3, erp:PinHeader_1x03_P2.54mm_Vertical, symbol erp:Conn_01x03_Male
Connections:
- wire segments 411 -> 415
Other:
- moved on the sheet: C8, D8, D9, Q7, R17, R19, R6

Commit message: Changed TVS diodes
Parts:
- D10, D11, D12, D13, D14, D15, D16, D17, D18, D28, D29, D3, D4, D5, D6, D7: value SMM4F15A -> SMA6F15AY; footprint (none) -> erp:D_SMA; symbol erp:D_TVS -> erp:D_Zener
Changed lines of the file:
@@
 Sheet 1 1
 Title "PowerUnit"
-Date "2019-12-02"
+Date "2019-12-03"
 Rev "A"
 Comp ""
@@
 	7250 950  7750 950
 $Comp
-L erp:D_TVS D12
+L erp:D_Zener D12
 U 1 1 5DAB9E3D
 P 6350 1050
 F 0 "D12" H 6350 1266 50  0000 C CNN
-F 1 "SMM4F15A" H 6350 1175 50  0000 C CNN
-F 2 "" H 6350 1050 50  0001 C CNN
+F 1 "SMA6F15AY" H 6350 1175 50  0000 C CNN
+F 2 "erp:D_SMA" H 6350 1050 50  0001 C CNN
 F 3 "" H 6350 1050 50  0001 C CNN
 F 4 "260001" H 6350 1050 50  0001 C CNN "ItemNo"
 	1    6350 1050
-	-1   0    0    1
+	1    0    0    1
 $EndComp
 $Comp
@@
 	6250 6550 6750 6550
 $Comp
-L erp:D_TVS D11
+L erp:D_Zener D11
 U 1 1 5DDB8481
 P 5350 6650
 F 0 "D11" H 5350 6866 50  0000 C CNN
-F 1 "SMM4F15A" H 5350 6775 50  0000 C CNN
-F 2 "" H 5350 6650 50  0001 C CNN
+F 1 "SMA6F15AY" H 5350 6775 50  0000 C CNN
+F 2 "erp:D_SMA" H 5350 6650 50  0001 C CNN
 F 3 "" H 5350 6650 50  0001 C CNN
 F 4 "260001" H 5350 6650 50  0001 C CNN "ItemNo"
 	1    5350 6650
-	-1   0    0    1
+	1    0    0    1
 $EndComp
 $Comp
@@
 	4150 6550 4650 6550
 $Comp
-L erp:D_TVS D3
+L erp:D_Zener D3
 U 1 1 5DDC73B1
 P 3250 6650
 F 0 "D3" H 3250 6866 50  0000 C CNN
-F 1 "SMM4F15A" H 3250 6775 50  0000 C CNN
-F 2 "" H 3250 6650 50  0001 C CNN
+F 1 "SMA6F15AY" H 3250 6775 50  0000 C CNN
+F 2 "erp:D_SMA" H 3250 6650 50  0001 C CNN
 F 3 "" H 3250 6650 50  0001 C CNN
 F 4 "260001" H 3250 6650 50  0001 C CNN "ItemNo"
 	1    3250 6650
-	-1   0    0    1
+	1    0    0    1
 $EndComp
 $Comp
@@
 	5150 950  5650 950
 $Comp
-L erp:D_TVS D4
+L erp:D_Zener D4
 U 1 1 5DE7B398
 P 4250 1050
 F 0 "D4" H 4250 1266 50  0000 C CNN
-F 1 "SMM4F15A" H 4250 1175 50  0000 C CNN
-F 2 "" H 4250 1050 50  0001 C CNN
+F 1 "SMA6F15AY" H 4250 1175 50  0000 C CNN
+F 2 "erp:D_SMA" H 4250 1050 50  0001 C CNN
 F 3 "" H 4250 1050 50  0001 C CNN
 F 4 "260001" H 4250 1050 50  0001 C CNN "ItemNo"
 	1    4250 1050
-	-1   0    0    1
+	1    0    0    1
 $EndComp
 $Comp
@@
 	7250 2050 7750 2050
 $Comp
-L erp:D_TVS D13
+L erp:D_Zener D13
 U 1 1 5DEE641F
 P 6350 2150
 F 0 "D13" H 6350 2366 50  0000 C CNN
-F 1 "SMM4F15A" H 6350 2275 50  0000 C CNN
-F 2 "" H 6350 2150 50  0001 C CNN
+F 1 "SMA6F15AY" H 6350 2275 50  0000 C CNN
+F 2 "erp:D_SMA" H 6350 2150 50  0001 C CNN
 F 3 "" H 6350 2150 50  0001 C CNN
 F 4 "260001" H 6350 2150 50  0001 C CNN "ItemNo"
 	1    6350 2150
-	-1   0    0    1
+	1    0    0    1
 $EndComp
 $Comp
@@
 	5150 2050 5650 2050
 $Comp
-L erp:D_TVS D5
+L erp:D_Zener D5
 U 1 1 5DF0D28B
 P 4250 2150
 F 0 "D5" H 4250 2366 50  0000 C CNN
-F 1 "SMM4F15A" H 4250 2275 50  0000 C CNN
-F 2 "" H 4250 2150 50  0001 C CNN
+F 1 "SMA6F15AY" H 4250 2275 50  0000 C CNN
+F 2 "erp:D_SMA" H 4250 2150 50  0001 C CNN
 F 3 "" H 4250 2150 50  0001 C CNN
 F 4 "260001" H 4250 2150 50  0001 C CNN "ItemNo"
 	1    4250 2150
-	-1   0    0    1
+	1    0    0    1
 $EndComp
 $Comp
@@
 OUT_BRAKE_A
 $Comp
-L erp:D_TVS D7
+L erp:D_Zener D7
 U 1 1 5E11CA08
 P 4250 4350
 F 0 "D7" H 4250 4566 50  0000 C CNN
-F 1 "SMM4F15A" H 4250 4475 50  0000 C CNN
-F 2 "" H 4250 4350 50  0001 C CNN
+F 1 "SMA6F15AY" H 4250 4475 50  0000 C CNN
+F 2 "erp:D_SMA" H 4250 4350 50  0001 C CNN
 F 3 "" H 4250 4350 50  0001 C CNN
 F 4 "260001" H 4250 4350 50  0001 C CNN "ItemNo"
 	1    4250 4350
-	-1   0    0    1
+	1    0    0    1
 $EndComp
 $Comp
@@
 	7250 4250 7750 4250
 $Comp
-L erp:D_TVS D15
+L erp:D_Zener D15
 U 1 1 5E13DE65
 P 6350 4350
 F 0 "D15" H 6350 4566 50  0000 C CNN
-F 1 "SMM4F15A" H 6350 4475 50  0000 C CNN
-F 2 "" H 6350 4350 50  0001 C CNN
+F 1 "SMA6F15AY" H 6350 4475 50  0000 C CNN
+F 2 "erp:D_SMA" H 6350 4350 50  0001 C CNN
 F 3 "" H 6350 4350 50  0001 C CNN
 F 4 "260001" H 6350 4350 50  0001 C CNN "ItemNo"
 	1    6350 4350
-	-1   0    0    1
+	1    0    0    1
 $EndComp
 $Comp
@@
 	6500 5300 7000 5300
 $Comp
-L erp:D_TVS D10
+L erp:D_Zener D10
 U 1 1 5E23A064
 P 5600 5400
 F 0 "D10" H 5600 5616 50  0000 C CNN
-F 1 "SMM4F15A" H 5600 5525 50  0000 C CNN
-F 2 "" H 5600 5400 50  0001 C CNN
+F 1 "SMA6F15AY" H 5600 5525 50  0000 C CNN
+F 2 "erp:D_SMA" H 5600 5400 50  0001 C CNN
 F 3 "" H 5600 5400 50  0001 C CNN
 F 4 "260001" H 5600 5400 50  0001 C CNN "ItemNo"
 	1    5600 5400
-	-1   0    0    1
+	1    0    0    1
 $EndComp
 $Comp
@@
 	5150 3150 5650 3150
 $Comp
-L erp:D_TVS D6
+L erp:D_Zener D6
 U 1 1 5E23A0A7
 P 4250 3250
 F 0 "D6" H 4250 3466 50  0000 C CNN
-F 1 "SMM4F15A" H 4250 3375 50  0000 C CNN
-F 2 "" H 4250 3250 50  0001 C CNN
+F 1 "SMA6F15AY" H 4250 3375 50  0000 C CNN
+F 2 "erp:D_SMA" H 4250 3250 50  0001 C CNN
 F 3 "" H 4250 3250 50  0001 C CNN
 F 4 "260001" H 4250 3250 50  0001 C CNN "ItemNo"
 	1    4250 3250
-	-1   0    0    1
+	1    0    0    1
 $EndComp
 $Comp
@@
 $EndComp
 $Comp
-L erp:D_TVS D28
+L erp:D_Zener D28
 U 1 1 5E04DBEE
 P 9800 5600
 F 0 "D28" H 9800 5816 50  0000 C CNN
-F 1 "SMM4F15A" H 9800 5725 50  0000 C CNN
-F 2 "" H 9800 5600 50  0001 C CNN
+F 1 "SMA6F15AY" H 9800 5725 50  0000 C CNN
+F 2 "erp:D_SMA" H 9800 5600 50  0001 C CNN
 F 3 "" H 9800 5600 50  0001 C CNN
 F 4 "260001" H 9800 5600 50  0001 C CNN "ItemNo"
@@
 $EndComp
 $Comp
-L erp:D_TVS D29
+L erp:D_Zener D29
 U 1 1 5E2C2953
 P 9900 1150
 F 0 "D29" H 9900 1366 50  0000 C CNN
-F 1 "SMM4F15A" H 9900 1275 50  0000 C CNN
-F 2 "" H 9900 1150 50  0001 C CNN
+F 1 "SMA6F15AY" H 9900 1275 50  0000 C CNN
+F 2 "erp:D_SMA" H 9900 1150 50  0001 C CNN
 F 3 "" H 9900 1150 50  0001 C CNN
 F 4 "260001" H 9900 1150 50  0001 C CNN "ItemNo"
@@
 $EndComp
 $Comp
-L erp:D_TVS D17
+L erp:D_Zener D17
 U 1 1 5E30DA3F
 P 8400 4450
 F 0 "D17" H 8400 4666 50  0000 C CNN
-F 1 "SMM4F15A" H 8400 4575 50  0000 C CNN
-F 2 "" H 8400 4450 50  0001 C CNN
+F 1 "SMA6F15AY" H 8400 4575 50  0000 C CNN
+F 2 "erp:D_SMA" H 8400 4450 50  0001 C CNN
 F 3 "" H 8400 4450 50  0001 C CNN
 F 4 "260001" H 8400 4450 50  0001 C CNN "ItemNo"
@@
 $EndComp
 $Comp
-L erp:D_TVS D16
+L erp:D_Zener D16
 U 1 1 5E35A899
 P 8400 3350
 F 0 "D16" H 8400 3566 50  0000 C CNN
-F 1 "SMM4F15A" H 8400 3475 50  0000 C CNN
-F 2 "" H 8400 3350 50  0001 C CNN
+F 1 "SMA6F15AY" H 8400 3475 50  0000 C CNN
+F 2 "erp:D_SMA" H 8400 3350 50  0001 C CNN
 F 3 "" H 8400 3350 50  0001 C CNN
 F 4 "260001" H 8400 3350 50  0001 C CNN "ItemNo"
@@
 	7250 3150 7750 3150
 $Comp
-L erp:D_TVS D14
+L erp:D_Zener D14
 U 1 1 5DF3A899
 P 6350 3250
 F 0 "D14" H 6350 3466 50  0000 C CNN
-F 1 "SMM4F15A" H 6350 3375 50  0000 C CNN
-F 2 "" H 6350 3250 50  0001 C CNN
+F 1 "SMA6F15AY" H 6350 3375 50  0000 C CNN
+F 2 "erp:D_SMA" H 6350 3250 50  0001 C CNN
 F 3 "" H 6350 3250 50  0001 C CNN
 F 4 "260001" H 6350 3250 50  0001 C CNN "ItemNo"
 	1    6350 3250
-	-1   0    0    1
+	1    0    0    1
 $EndComp
 $Comp
@@
 $EndComp
 $Comp
-L erp:D_TVS D18
+L erp:D_Zener D18
 U 1 1 5E1611A8
 P 8400 1150
 F 0 "D18" H 8400 1366 50  0000 C CNN
-F 1 "SMM4F15A" H 8400 1275 50  0000 C CNN
-F 2 "" H 8400 1150 50  0001 C CNN
+F 1 "SMA6F15AY" H 8400 1275 50  0000 C CNN
+F 2 "erp:D_SMA" H 8400 1150 50  0001 C CNN
 F 3 "" H 8400 1150 50  0001 C CNN
 F 4 "260001" H 8400 1150 50  0001 C CNN "ItemNo"

Commit message: All footprints added
Parts:
- removed J4: REDCUBE, symbol erp:Conn_02x05_Top_Bottom
- added J4: REDCUBE, erp:Wurth_WP-BUCF_M6, symbol erp:Conn_02x08_Top_Bottom
- F1, F2, F3, F4, F5, F6, F7, F8: footprint (none) -> erp:Keystone_FuseHolder
- J1, J2: footprint (none) -> erp:Molex_MX150_2x10_Header
- J3: footprint (none) -> erp:Molex_MX150_2x04_Header
- Q10, Q11, Q12, Q13, Q2, Q3, Q4, Q5, Q6, Q7, Q9: symbol erp:Q_PMOS_GDSD -> erp:Q_PMOS_GDS
Connections:
- net +12V: now also J4.1 (Pin_1), J4.10 (Pin_10), J4.11 (Pin_11), J4.12 (Pin_12), J4.13 (Pin_13), J4.14 (Pin_14), J4.15 (Pin_15), J4.16 (Pin_16), J4.2 (Pin_2), J4.3 (Pin_3), J4.4 (Pin_4), J4.5 (Pin_5), J4.6 (Pin_6), J4.7 (Pin_7), J4.8 (Pin_8), J4.9 (Pin_9)
- net OUT_AUX: no longer Q4.4 (D)
- net OUT_BRAKE_A: no longer Q6.4 (D)
- net OUT_BRAKE_B: no longer Q13.4 (D)
- net OUT_FUEL: no longer Q11.4 (D)
- net OUT_IGN: no longer Q10.4 (D)
- net OUT_INJECT: no longer Q3.4 (D)
- net OUT_LEFT: no longer Q2.4 (D)
- net OUT_LIGHT: no longer Q12.4 (D)
- net OUT_RAIN: no longer Q5.4 (D)
- net OUT_RIGHT: no longer Q9.4 (D)
Changed lines of the file:
@@
 Sheet 1 1
 Title "PowerUnit"
-Date "2019-12-03"
+Date "2019-12-04"
 Rev "A"
 Comp ""
@@
 F 0 "J1" H 1650 1817 50  0000 C CNN
 F 1 "MX150-20" H 1650 1726 50  0000 C CNN
-F 2 "" H 1600 1200 50  0001 C CNN
+F 2 "erp:Molex_MX150_2x10_Header" H 1600 1200 50  0001 C CNN
 F 3 "" H 1600 1200 50  0001 C CNN
 F 4 "501000" H 1600 1200 50  0001 C CNN "ItemNo"
@@
 F 0 "J2" H 1650 3117 50  0000 C CNN
 F 1 "MX150-20" H 1650 3026 50  0000 C CNN
-F 2 "" H 1600 2500 50  0001 C CNN
+F 2 "erp:Molex_MX150_2x10_Header" H 1600 2500 50  0001 C CNN
 F 3 "" H 1600 2500 50  0001 C CNN
 F 4 "501000" H 1600 2500 50  0001 C CNN "ItemNo"
@@
 F 0 "F6" V 8953 1900 50  0000 C CNN
 F 1 "FUSE" V 9044 1900 50  0000 C CNN
-F 2 "" V 9080 1900 50  0001 C CNN
+F 2 "erp:Keystone_FuseHolder" V 9080 1900 50  0001 C CNN
 F 3 "" H 9150 1900 50  0001 C CNN
 F 4 "401000" H 9150 1900 50  0001 C CNN "ItemNo"
@@
 F 0 "F1" V 10453 800 50  0000 C CNN
 F 1 "FUSE" V 10544 800 50  0000 C CNN
-F 2 "" V 10580 800 50  0001 C CNN
+F 2 "erp:Keystone_FuseHolder" V 10580 800 50  0001 C CNN
 F 3 "" H 10650 800 50  0001 C CNN
 F 4 "401000" H 10650 800 50  0001 C CNN "ItemNo"
@@
 F 0 "F2" V 10453 1900 50  0000 C CNN
 F 1 "FUSE" V 10544 1900 50  0000 C CNN
-F 2 "" V 10580 1900 50  0001 C CNN
+F 2 "erp:Keystone_FuseHolder" V 10580 1900 50  0001 C CNN
 F 3 "" H 10650 1900 50  0001 C CNN
 F 4 "401000" H 10650 1900 50  0001 C CNN "ItemNo"
@@
 	10200 2000 9800 2000
 $Comp
-L erp:Q_PMOS_GDSD Q10
+L erp:Q_PMOS_GDS Q10
 U 1 1 5DD64F7C
 P 6950 1050
@@
 	0    1    1    0
 $EndComp
-Wire Wire Line
-	6750 950  6650 950
-Wire Wire Line
-	6750 850  6650 850
-Wire Wire Line
-	6650 850  6650 950
-Connection ~ 6650 950
 Text Label 7750 950  2    50   ~ 0
 PWD_IGN
@@
 Connection ~ 6150 950
 Wire Wire Line
-	6150 950  6650 950
-Wire Wire Line
 	5950 950  6150 950
 Wire Wire Line
@@
 IN_IGN
 $Comp
-L erp:Q_PMOS_GDSD Q9
+L erp:Q_PMOS_GDS Q9
 U 1 1 5DDB844E
 P 5950 6650
@@
 	0    1    1    0
 $EndComp
-Wire Wire Line
-	5750 6550 5650 6550
-Wire Wire Line
-	5750 6450 5650 6450
-Wire Wire Line
-	5650 6450 5650 6550
-Connection ~ 5650 6550
 Text Label 6750 6550 2    50   ~ 0
 PWD_LIGHT
@@
 Connection ~ 5150 6550
 Wire Wire Line
-	5150 6550 5650 6550
-Wire Wire Line
 	4950 6550 5150 6550
 Wire Wire Line
@@
 MCU_OUT_RIGHT
 $Comp
-L erp:Q_PMOS_GDSD Q2
+L erp:Q_PMOS_GDS Q2
 U 1 1 5DDC737E
 P 3850 6650
@@
 	0    1    1    0
 $EndComp
-Wire Wire Line
-	3650 6550 3550 6550
-Wire Wire Line
-	3650 6450 3550 6450
-Wire Wire Line
-	3550 6450 3550 6550
-Connection ~ 3550 6550
 Text Label 4650 6550 2    50   ~ 0
 PWD_LIGHT
@@
 Connection ~ 3050 6550
 Wire Wire Line
-	3050 6550 3550 6550
-Wire Wire Line
 	2850 6550 3050 6550
 Wire Wire Line
@@
 OUT_INJECT
 $Comp
-L erp:Q_PMOS_GDSD Q3
+L erp:Q_PMOS_GDS Q3
 U 1 1 5DE7B377
 P 4850 1050
@@
 	0    1    1    0
 $EndComp
-Wire Wire Line
-	4650 950  4550 950
-Wire Wire Line
-	4650 850  4550 850
-Wire Wire Line
-	4550 850  4550 950
-Connection ~ 4550 950
 Text Label 5650 950  2    50   ~ 0
 PWD_INJECT
@@
 Connection ~ 4050 950
 Wire Wire Line
-	4050 950  4550 950
-Wire Wire Line
 	3850 950  4050 950
 Wire Wire Line
@@
 F 0 "F3" V 10453 3000 50  0000 C CNN
 F 1 "FUSE" V 10544 3000 50  0000 C CNN
-F 2 "" V 10580 3000 50  0001 C CNN
+F 2 "erp:Keystone_FuseHolder" V 10580 3000 50  0001 C CNN
 F 3 "" H 10650 3000 50  0001 C CNN
 F 4 "401000" H 10650 3000 50  0001 C CNN "ItemNo"
@@
 F 0 "F4" V 10453 4100 50  0000 C CNN
 F 1 "FUSE" V 10544 4100 50  0000 C CNN
-F 2 "" V 10580 4100 50  0001 C CNN
+F 2 "erp:Keystone_FuseHolder" V 10580 4100 50  0001 C CNN
 F 3 "" H 10650 4100 50  0001 C CNN
 F 4 "401000" H 10650 4100 50  0001 C CNN "ItemNo"
@@
 	10200 4200 9800 4200
 $Comp
-L erp:Q_PMOS_GDSD Q11
+L erp:Q_PMOS_GDS Q11
 U 1 1 5DEE63FE
 P 6950 2150
@@
 	0    1    1    0
 $EndComp
-Wire Wire Line
-	6750 2050 6650 2050
-Wire Wire Line
-	6750 1950 6650 1950
-Wire Wire Line
-	6650 1950 6650 2050
-Connection ~ 6650 2050
 Text Label 7750 2050 2    50   ~ 0
 PWD_FUEL
@@
 Connection ~ 6150 2050
 Wire Wire Line
-	6150 2050 6650 2050
-Wire Wire Line
 	5950 2050 6150 2050
 Wire Wire Line
@@
 OUT_FUEL
 $Comp
-L erp:Q_PMOS_GDSD Q4
+L erp:Q_PMOS_GDS Q4
 U 1 1 5DF0D26A
 P 4850 2150
@@
 	0    1    1    0
 $EndComp
-Wire Wire Line
-	4650 2050 4550 2050
-Wire Wire Line
-	4650 1950 4550 1950
-Wire Wire Line
-	4550 1950 4550 2050
-Connection ~ 4550 2050
 Text Label 5650 2050 2    50   ~ 0
 PWD_AUX
@@
 Connection ~ 4050 2050
 Wire Wire Line
-	4050 2050 4550 2050
-Wire Wire Line
 	3850 2050 4050 2050
 Wire Wire Line
@@
 F 0 "F5" V 8953 800 50  0000 C CNN
 F 1 "FUSE" V 9044 800 50  0000 C CNN
-F 2 "" V 9080 800 50  0001 C CNN
+F 2 "erp:Keystone_FuseHolder" V 9080 800 50  0001 C CNN
 F 3 "" H 9150 800 50  0001 C CNN
 F 4 "401000" H 9150 800 50  0001 C CNN "ItemNo"
@@
 F 0 "F7" V 8953 3000 50  0000 C CNN
 F 1 "FUSE" V 9044 3000 50  0000 C CNN
-F 2 "" V 9080 3000 50  0001 C CNN
+F 2 "erp:Keystone_FuseHolder" V 9080 3000 50  0001 C CNN
 F 3 "" H 9150 3000 50  0001 C CNN
 F 4 "401000" H 9150 3000 50  0001 C CNN "ItemNo"
@@
 F 0 "F8" V 8953 4100 50  0000 C CNN
 F 1 "FUSE" V 9044 4100 50  0000 C CNN
-F 2 "" V 9080 4100 50  0001 C CNN
+F 2 "erp:Keystone_FuseHolder" V 9080 4100 50  0001 C CNN
 F 3 "" H 9150 4100 50  0001 C CNN
 F 4 "401000" H 9150 4100 50  0001 C CNN "ItemNo"
@@
 	5450 7150 5650 7150
 $Comp
-L erp:Q_PMOS_GDSD Q6
+L erp:Q_PMOS_GDS Q6
 U 1 1 5E11C9E7
 P 4850 4350
@@
 	0    1    1    0
 $EndComp
-Wire Wire Line
-	4650 4250 4550 4250
-Wire Wire Line
-	4650 4150 4550 4150
-Wire Wire Line
-	4550 4150 4550 4250
-Connection ~ 4550 4250
 Text Label 5650 4250 2    50   ~ 0
 PWD_LIGHT
@@
 Connection ~ 4050 4250
 Wire Wire Line
-	4050 4250 4550 4250
-Wire Wire Line
 	3850 4250 4050 4250
 Wire Wire Line
@@
 	4350 4850 4850 4850
 $Comp
-L erp:Q_PMOS_GDSD Q13
+L erp:Q_PMOS_GDS Q13
 U 1 1 5E13DE45
 P 6950 4350
@@
 Wire Wire Line
 	7150 4250 7250 4250
-Wire Wire Line
-	6750 4250 6650 4250
-Wire Wire Line
-	6650 4150 6650 4250
-Connection ~ 6650 4250
 Text Label 7750 4250 2    50   ~ 0
 PWD_MISC
@@
 Connection ~ 6150 4250
 Wire Wire Line
-	6150 4250 6650 4250
-Wire Wire Line
 	5950 4250 6150 4250
 Wire Wire Line
@@
 Connection ~ 7250 4550
 Wire Wire Line
-	6750 4150 6650 4150
-Wire Wire Line
 	5050 4250 5650 4250
 Wire Wire Line
@@
 Connection ~ 4850 4850
 $Comp
-L erp:Q_PMOS_GDSD Q7
+L erp:Q_PMOS_GDS Q7
 U 1 1 5E23A043
 P 6200 5400
@@
 	0    1    1    0
 $EndComp
-Wire Wire Line
-	6000 5300 5900 5300
-Wire Wire Line
-	5650 5150 5550 5150
-Wire Wire Line
-	5900 5200 5900 5300
-Connection ~ 5900 5300
 Text Label 7000 5300 2    50   ~ 0
 PWD_FAN
@@
 Connection ~ 5400 5300
 Wire Wire Line
-	5400 5300 5900 5300
-Wire Wire Line
 	5200 5300 5400 5300
 Wire Wire Line
@@
 	5700 5900 6200 5900
 $Comp
-L erp:Q_PMOS_GDSD Q5
+L erp:Q_PMOS_GDS Q5
 U 1 1 5E23A086
 P 4850 3250
@@
 	0    1    1    0
 $EndComp
-Wire Wire Line
-	4650 3150 4550 3150
-Wire Wire Line
-	4650 3050 4550 3050
-Wire Wire Line
-	4550 3050 4550 3150
-Connection ~ 4550 3150
 Text Label 5650 3150 2    50   ~ 0
 PWD_MISC
@@
 Connection ~ 4050 3150
 Wire Wire Line
-	4050 3150 4550 3150
-Wire Wire Line
 	3850 3150 4050 3150
 Wire Wire Line
@@
 F 0 "J3" H 1650 3817 50  0000 C CNN
 F 1 "MX150-8" H 1650 3726 50  0000 C CNN
-F 2 "" H 1600 3500 50  0001 C CNN
+F 2 "erp:Molex_MX150_2x04_Header" H 1600 3500 50  0001 C CNN
 F 3 "" H 1600 3500 50  0001 C CNN
 F 4 "501001" H 1600 3500 50  0001 C CNN "ItemNo"
@@
 OUT_RAIN
 $Comp
-L erp:Conn_02x05_Top_Bottom J4
-U 1 1 5E50F8BC
-P 10450 5750
-F 0 "J4" H 10500 6167 50  0000 C CNN
-F 1 "REDCUBE" H 10500 6076 50  0000 C CNN
-F 2 "" H 10450 5750 50  0001 C CNN
-F 3 "" H 10450 5750 50  0001 C CNN
-F 4 "502000" H 10450 5750 50  0001 C CNN "ItemNo"
-	1    10450 5750
-	1    0    0    -1
-$EndComp
-$Comp
 L erp:L5150BN U2
 U 1 1 5E510AC6
@@
 IN_RIGHT
 $Comp
-L erp:Q_PMOS_GDSD Q12
+L erp:Q_PMOS_GDS Q12
 U 1 1 5DF3A878
 P 6950 3250
@@
 	0    1    1    0
 $EndComp
-Wire Wire Line
-	6750 3150 6650 3150
-Wire Wire Line
-	6750 3050 6650 3050
-Wire Wire Line
-	6650 3050 6650 3150
-Connection ~ 6650 3150
 Text Label 7750 3150 2    50   ~ 0
 PWD_LIGHT
@@
 Connection ~ 6150 3150
 Wire Wire Line
-	6150 3150 6650 3150
-Wire Wire Line
 	5950 3150 6150 3150
 Wire Wire Line
@@
 	3100 5250 3100 5450
 Connection ~ 3100 5250
+$Comp
+L erp:Conn_02x08_Top_Bottom J4
+U 1 1 5DF2B301
+P 10450 5850
+F 0 "J4" H 10500 6367 50  0000 C CNN
+F 1 "REDCUBE" H 10500 6276 50  0000 C CNN
+F 2 "erp:Wurth_WP-BUCF_M6" H 10450 5850 50  0001 C CNN
+F 3 "" H 10450 5850 50  0001 C CNN
+F 4 "502000" H 10450 5850 50  0001 C CNN "ItemNo"
+	1    10450 5850
+	1    0    0    -1
+$EndComp
+Wire Wire Line
+	10250 6050 10150 6050
+Wire Wire Line
+	10150 6050 10150 5950
+Connection ~ 10150 5950
+Wire Wire Line
+	10250 6150 10150 6150
+Wire Wire Line
+	10150 6150 10150 6050
+Connection ~ 10150 6050
+Wire Wire Line
+	10250 6250 10150 6250
+Wire Wire Line
+	10150 6250 10150 6150
+Connection ~ 10150 6150
+Wire Wire Line
+	10750 6050 10850 6050
+Wire Wire Line
+	10850 6050 10850 5950
+Connection ~ 10850 5950
+Wire Wire Line
+	10750 6150 10850 6150
+Wire Wire Line
+	10850 6150 10850 6050
+Connection ~ 10850 6050
+Wire Wire Line
+	10750 6250 10850 6250
+Wire Wire Line
+	10850 6250 10850 6150
+Connection ~ 10850 6150
+Wire Wire Line
+	4050 950  4650 950
+Wire Wire Line
+	6150 950  6750 950
+Wire Wire Line
+	6150 2050 6750 2050
+Wire Wire Line
+	4050 2050 4650 2050
+Wire Wire Line
+	6150 3150 6750 3150
+Wire Wire Line
+	4050 3150 4650 3150
+Wire Wire Line
+	4050 4250 4650 4250
+Wire Wire Line
+	6150 4250 6750 4250
+Wire Wire Line
+	5400 5300 6000 5300
+Wire Wire Line
+	5150 6550 5750 6550
+Wire Wire Line
+	3050 6550 3650 6550
 $EndSCHEMATC

Commit message: First PCB Layout done
Parts:
- removed D16, D18: SMA6F15AY, erp:D_SMA, symbol erp:D_Zener
- added D38, D43: SMA6F15AY, erp:D_SMA, symbol erp:D_Zener
- added D39, D41: LL4148, erp:D_MiniMELF, symbol erp:D
- added D40, D42: RED, erp:LED_0805_2012Metric, symbol erp:LED
- added F1, F7: FUSE, erp:Keystone_FuseHolder, symbol erp:Fuse_T2
- added J10, J11, J12, J13, J6, J7, J8, J9: MH_M4, erp:MountingHole_4.3mm_M4_Pad_Via, symbol erp:Conn_01x01
- added R37, R38, R39: 2.2k, erp:R_0805_2012Metric, symbol erp:R
- renumbered F4 to F10, F1 to F2, F2 to F4, F8 to F6, F6 to F8, F7 to F9
Connections:
- net +12V: now also D40.2 (A), D42.2 (A), F1.1A, F1.1B, F7.1A, F7.1B
- net +5V: now also R1.1, R3.1
- net GND: now also J1.1 (Pin_1), J2.1 (Pin_1), J3.1 (Pin_1), D38.2 (A), D43.2 (A), J10.1 (Pin_1), J11.1 (Pin_1), J12.1 (Pin_1), J13.1 (Pin_1), J6.1 (Pin_1), J7.1 (Pin_1), J8.1 (Pin_1), J9.1 (Pin_1), R37.2, R38.2; no longer J1.11 (Pin_11), J2.11 (Pin_11), J3.5 (Pin_5)
- net IN_AUX: now also J2.5 (Pin_5); no longer J2.6 (Pin_6)
- net IN_FAN_A: now also J1.14 (Pin_14); no longer J1.15 (Pin_15)
- net IN_FAN_B: now also J2.17 (Pin_17); no longer J2.15 (Pin_15)
- net IN_FUEL: now also J2.15 (Pin_15); no longer J2.17 (Pin_17)
- net IN_IGN: now also J2.18 (Pin_18); no longer J2.19 (Pin_19)
- net IN_INJECT: now also J1.15 (Pin_15); no longer J1.14 (Pin_14)
- net IN_LIGHT: now also J2.16 (Pin_16); no longer J2.18 (Pin_18)
- net IN_RAIN: now also J2.14 (Pin_14); no longer J2.16 (Pin_16)
- net OUT_AUX: now also J2.9 (Pin_9); no longer J2.5 (Pin_5)
- net OUT_BRAKE_A: now also J3.8 (Pin_8); no longer J3.6 (Pin_6)
- net OUT_BRAKE_B: now also J3.3 (Pin_3); no longer J3.7 (Pin_7)
- net OUT_FUEL: now also J3.4 (Pin_4); no longer J3.8 (Pin_8)
- net OUT_LEFT: now also J2.2 (Pin_2), J3.6 (Pin_6); no longer J2.8 (Pin_8), J3.2 (Pin_2)
- net OUT_LIGHT: now also J1.6 (Pin_6), J2.4 (Pin_4), J3.5 (Pin_5); no longer J1.18 (Pin_18), J2.3 (Pin_3), J3.1 (Pin_1)
- net OUT_RAIN: now also J3.2 (Pin_2); no longer J3.4 (Pin_4)
- net OUT_RIGHT: now also J2.3 (Pin_3), J3.7 (Pin_7); no longer J2.9 (Pin_9), J3.3 (Pin_3)
- net PWD_AUX: now also J2.8 (Pin_8); no longer J2.2 (Pin_2)
- net PWD_ECU: now also J1.7 (Pin_7), J1.8 (Pin_8); no longer J1.6 (Pin_6), J2.4 (Pin_4)
- net PWD_FAN: no longer J1.9 (Pin_9)
- net PWD_LIGHT: now also R39.1; no longer R1.1, R3.1
- net PWD_MISC: no longer J2.7 (Pin_7)
- net START: now also J1.18 (Pin_18), J1.19 (Pin_19), J2.19 (Pin_19); no longer J1.7 (Pin_7), J1.8 (Pin_8), J2.14 (Pin_14)
- net at C13.1, Q13.1 (G), Q6.1 (G)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: now also R39.2
- new net: D41.1 (K), D42.1 (K), R38.1
- new net: D39.1 (K), D40.1 (K), R37.1
- new net PWD_DASH: D38.1 (K), D39.2 (A), F7.2A, F7.2B, J2.6 (Pin_6), J2.7 (Pin_7)
- new net PWD_START: D41.2 (A), D43.1 (K), F1.2A, F1.2B, J1.9 (Pin_9)
- no-connect marks 4 -> 3
Other:
- moved on the sheet: C1, C14, C15, C3, C4, C5, C6, C7, C8, C9, D10, D11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
