File: PCB/PowerUnit.kicad_sch (KiCad schematic)
At the start: 119 parts, among them J1 MX150-20, J2 MX150-20, J3 MX150-8, J4 REDCUBE, J5 REDFIT-4, Q1 BC847C, Q2 BC847C, U1 STM8S001J3M3, U10 BTS6143D, U11 BTS6143D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

Commit message: Add Fan pull-up
Parts:
- added R8: 1k, erp:R_0805_2012Metric, symbol erp:R
Connections:
- net PWD_FAN: now also R8.2
- net at D8.2 (A), D9.2 (A), R17.2: now also R8.1

Commit message: Production data Rev C
Parts:
- added C5: 100n, erp:C_0805_2012Metric, symbol erp:C
- added Q3: BC847C, erp:SOT-23, symbol erp:Q_NPN_BEC
- added R14, R15: 1k, erp:R_0805_2012Metric, symbol erp:R
- D10, D11, D12, D13, D14, D15, D17, D28, D29, D3, D38, D4, D43, D5, D6, D7: value SMA6F15AY -> SM6F15AY; footprint erp:D_SMA -> erp:D_SOD-128; ItemNo 260001 -> 260003
Connections:
- net GND: now also C5.2, Q3.2 (E), R14.1
- net IN_FAN_P: now reaches J1.12 (Pin_12)
- net IN_FAN_P: now also R14.2, R15.2
- net at D8.2 (A), D9.2 (A), R17.2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: now also Q3.3 (C)
- new net: C5.1, Q3.1 (B), R15.1
- no-connect marks 15 -> 14
Other:
- moved on the sheet: D11, D3, D8, D9, Q1, Q2, R13, R18, R5, R7, U12, U13

Commit message: Update Assembly data to Rev C
Parts:
- R6: now not fitted
Changed lines of the file:
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@@
   )
   (symbol (lib_id "erp:R") (at 60.96 128.27 0) (unit 1)
-    (in_bom yes) (on_board yes) (dnp no)
+    (in_bom yes) (on_board yes) (dnp yes)
     (property "Reference" "R6" (at 62.738 127.1016 0)
       (effects (font (size 1.27 1.27)) (justify left))
